File: KiCadProjects/PowerSupply/PowerSupply.sch (KiCad schematic (older format))
At the start: 36 parts

Commit message: More power suppply edits
Parts:
- removed J?: USB_C_Receptacle_USB2.0, symbol Connector:USB_C_Receptacle_USB2.0
- added C107, C108, C? (x2): 4u7, symbol Device:C
- added C109, C110: 100n, symbol Device:C
- added J103: Screw_Terminal_01x04, symbol Connector:Screw_Terminal_01x04
- added J104: Screw_Terminal_01x05, symbol Connector:Screw_Terminal_01x07
- added J?: 213716-0001, Molex-213716-0001-*, symbol MOLEX_USB_C_213716-0001:213716-0001
- J101: renamed from J?; footprint (none) -> Connector_JST:JST_EH_B2B-EH-A_1x02_P2.50mm_Vertical
- U102: renamed from U?; symbol eec:MCP73832T-2ACI_OT -> MCP7382T:MCP73832T-2ACI_OT
- gave numbers to parts that had none: 33
Connections:
- wire segments 125 -> 170
- no-connect marks 14 -> 10
Other:
- note added: "LM2735X has min duty cycle of 5%,\nso when USB is connected, \n+5V will be approximately 5.26V. \nThis should be fine as it is regulated\nto 3.3V on the Teensy which will \nbe used for most other circuits"
- note added: "To Main PCB"
- note added: "To SiPm PCB"
- moved on the sheet: C102, C103, C104, C105, C106, D101, D102, D103, J101, L101, R108, R109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

Commit message: updated schematic
Parts:
- removed C101: 4.7u, symbol Device:C
- removed C102, C106, C? (x2): 4u7, symbol Device:C
- removed C103, C105: 10u, symbol Device:C
- removed C104: 1.8n, symbol Device:C
- removed C111, C112: C, symbol Device:C
- removed D101, D102, D103, D104: D_Schottky, symbol Device:D_Schottky
- removed J101: Conn_01x02, Connector_JST:JST_EH_B2B-EH-A_1x02_P2.50mm_Vertical, symbol Connector_Generic:Conn_01x02
- removed J?: 213716-0001, Molex-213716-0001-*, symbol MOLEX_USB_C_213716-0001:213716-0001
- removed L101: 3.9u, symbol pspice:INDUCTOR
- removed L102: 47u, symbol pspice:INDUCTOR
- removed R101, R102: 100K, symbol Device:R
- removed R103: 1K35, symbol Device:R
- removed R104, R108, R111: 10K, symbol Device:R
- removed R105: 6K98, symbol Device:R
- removed R106, R107: 1K, symbol Device:R
- removed R109: 10k, symbol Device:R
- removed R110: 9K, symbol Device:R
- removed R112: 30K, symbol Device:R
- removed R113, R114, R115: R, symbol Device:R
- removed U101: AD8541ARZ, SOIC127P600X175-8N, symbol AD8541ARZ:AD8541ARZ
- removed U102: MCP73832T-2ACI_OT, Microchip-C04-091-OT-0-F-*, symbol MCP7382T:MCP73832T-2ACI_OT
- removed U103: LM2735XMF, Package_TO_SOT_SMD:SOT-23-5, symbol Regulator_Switching:LM2735XMF
- removed U104: OP184FSZ, SOIC127P600X175-8N, symbol OP184FSZ:OP184FSZ
- removed U105: MAX5026EUT+T, SOT95P280X145-6N, symbol MAX5026EUT_T:MAX5026EUT+T
- C107, C108: footprint (none) -> Capacitor_SMD:C_1206_3216Metric
- C109, C110: footprint (none) -> Capacitor_SMD:C_0805_2012Metric
- J103: footprint (none) -> TerminalBlock_Phoenix:TerminalBlock_Phoenix_MKDS-1,5-4-5.08_1x04_P5.08mm_Horizontal
- J104: footprint (none) -> TerminalBlock_Phoenix:TerminalBlock_Phoenix_MKDS-1,5-5-5.08_1x05_P5.08mm_Horizontal
Connections:
- no-connect marks 10 -> 0
Other:
- note removed: "LM2735X has min duty cycle of 5%,\nso when USB is connected, \n+5V will be approximately 5.26V. \nThis should be fine as it is regulated\nto 3.3V on the Teensy which will \nbe used for most other circuits"
- moved on the sheet: C107, C108, C109, C110, J103, J104
