File: KiCadProjects/MainBoard/MainBoard/barometer.sch (KiCad schematic (older format))
At the start: 0 parts

Commit message: Update to Main PCB Schematic
Parts:
- added C?: 10u, symbol Device:C
- added C?: 2.2n, symbol Device:C
- added C? (x2): 100n, symbol Device:C
- added R?: 59K, symbol Device:R
- added R?: 59K - DNP, symbol Device:R
- added R?: 100K, symbol Device:R
- added TP? (x4): TestPoint, symbol Connector:TestPoint
- added U?: KP236, symbol KP236:KP236
Connections:
- net labels added: +5V, GND, PRESSURE_SENSE_NS
- wire segments 0 -> 34
Other:
- note added: "0.5\n"
- note added: "115"
- note added: "4.5"
- note added: "40"
- note added: "Pins 1-4 are used for\ntesting/calibrating and\nshould usually be left floating\n"
- note added: "Populate Pull-up\nor Pull-down res.\nNOT BOTH"
- note added: "Pressure [kPa]"
- note added: "VOUT = 0.01057*P[kPa]-0.32667"
- note added: "VOUT [V]"
